Commit message: updated

File: urdf/PiCar_urdf.urdf (robot description, URDF)
Before this commit: robot PiCar_urdf, 3 links, 2 joints
Links:
- link base_link: geometry collision mesh filename=package://ros2_picar/base_link.STL; visual mesh filename=package://ros2_picar/base_link.STL
- link laser_scan: geometry collision mesh filename=package://ros2_picar/laser_scan.STL; visual mesh filename=package://ros2_picar/laser_scan.STL
